File: d2000-minipc-io.kicad_sch (KiCad schematic)
At the start: 7 parts, among them J1 TX24-80R-LT-H1E, J2 USB_DEBUG, J3 USB3_A_Stacked, J4 USB3_A_Stacked, J5 HDMI_A, U1 CP2102N-Axx-xQFN24

Commit message: updated schematic
Parts:
- removed J3, J4: USB3_A_Stacked, symbol Connector:USB3_A_Stacked
- added C1, C13, C15, C16, C17, C18, C19, C2, C23, C24, C25, C26, C27, C28, C29, C3, C31, C32, C33, C34, C38, C4, C40, C42, C44, C5, C6, C7: 0.1uF, Capacitor_SMD:C_0402_1005Metric, symbol Device:C_Small
- added C10, C11, C56, C57: 22uF, Capacitor_SMD:C_0603_1608Metric, symbol Device:C_Small
- added C12, C14: 1000pF, Capacitor_SMD:C_0402_1005Metric, symbol Device:C_Small
- added C20, C21, C22: 1uF, Capacitor_SMD:C_0402_1005Metric, symbol Device:C_Small
- added C30, C35, C36, C37: 10uF, Capacitor_SMD:C_0603_1608Metric, symbol Device:C_Small
- added C39, C41, C43, C45: 150uF, Capacitor_SMD:C_Elec_4x5.4, symbol Device:C_Polarized_Small
- added C46, C47: 100nF, Capacitor_SMD:C_0402_1005Metric, symbol Device:C_Small
- added C48, C50, C59: 4.7uF, Capacitor_SMD:C_0603_1608Metric, symbol Device:C_Small
- added C49, C8: 1uF, Capacitor_SMD:C_0603_1608Metric, symbol Device:C_Small
- added C51, C52, C53, C54, C61, C62, C63, C64: 47uF, Capacitor_SMD:C_0603_1608Metric, symbol Device:C_Small
- added C55, C60: 0.1uF, Capacitor_SMD:C_0603_1608Metric, symbol Device:C_Small
- added C58, C9: 100nF, Capacitor_SMD:C_0603_1608Metric, symbol Device:C_Small
- added H1: MH_LEFT, MountingHole:MountingHole_3.2mm_M3_DIN965_Pad, symbol Mechanical:MountingHole_Pad
- added H2: MH_RIGHT, MountingHole:MountingHole_3.2mm_M3_DIN965_Pad, symbol Mechanical:MountingHole_Pad
- added J6: RJMG201K21120FR, RJMG201K21120FR:AMPHENOL_RJMG201K21120FR, symbol RJMG201K21120FR:RJMG201K21120FR
- added J8: DC_IN, DC-505:DC-505, symbol Connector:Jack-DC
- added L1, L2: 1.5uH, Inductor_SMD:L_TDK_VLP8040, symbol Device:L
- added R10, R11, R17: 1M, Resistor_SMD:R_0402_1005Metric, symbol Device:R_Small
- added R12, R25, R26, R32: 10k, Resistor_SMD:R_0603_1608Metric, symbol Device:R
- added R13, R22: 100k, Resistor_SMD:R_0603_1608Metric, symbol Device:R
- added R14: 9.53k, Resistor_SMD:R_0402_1005Metric, symbol Device:R_Small
- added R15, R16, R6, R7, R8, R9: 4.7k, Resistor_SMD:R_0402_1005Metric, symbol Device:R_Small
- added R18, R19, R4, R5: 4.7k, Resistor_SMD:R_0402_1005Metric, symbol Device:R
- added R2: 90.9k, Resistor_SMD:R_0402_1005Metric, symbol Device:R
- added R20, R21: 1.2k, Resistor_SMD:R_0402_1005Metric, symbol Device:R
- added R23, R30: 499k, Resistor_SMD:R_0603_1608Metric, symbol Device:R
- added R24, R33: ?, Resistor_SMD:R_0603_1608Metric, symbol Device:R
- added R27, R31: 2.2r, Resistor_SMD:R_0603_1608Metric, symbol Device:R_Small
- added R28, R29: 5.6k, Resistor_SMD:R_0402_1005Metric, symbol Device:R_Small
- added R3: 10k, Resistor_SMD:R_0402_1005Metric, symbol Device:R
- added U2: TUSB8041, Package_DFN_QFN:QFN-64-1EP_9x9mm_P0.5mm_EP6x6mm_ThermalVias, symbol Interface_USB:TUSB8041
- added U3, U4: TPS2561, Package_SON:VSON-10-1EP_3x3mm_P0.5mm_EP1.65x2.4mm_ThermalVias, symbol Interface_USB:TPS2561
- added U5, U6: SIC437A, Package_DFN_QFN:Vishay_PowerPAK_MLP44-24L_ThermalVias, symbol Regulator_Switching:SIC437A
- added USB1, USB2: USB-303WSD-BRY, XUNPU-USB-303WSD-BRY:USB-A-TH_XUNPU_USB-303WSD-BRY, symbol XUNPU-USB-303WSD-BRY:USB-303WSD-BRY
- added Y1: 24MHz, Crystal:Crystal_SMD_Abracon_ABM3B-4Pin_5.0x3.2mm, symbol Device:Crystal
- J1: value TX24-80R-LT-H1E -> TX24-80R; footprint CON80_2X40_MR_TX24_JAE -> TX24_80R_10ST_H1E:CON80_2X40_MU_TX24_JAE
- J2: footprint (none) -> Connector_USB:USB_C_Receptacle_HRO_TYPE-C-31-M-12
- J5: footprint (none) -> Connector_Video:HDMI_A_Molex_208658-1001_Horizontal
- U1: value CP2102N-Axx-xQFN24 -> CP2102N
Connections:
- net HDMI_DATA0_R is gone; now on net HDMI_DATA0_P: J1.21
- net 3V3: now also C23.2, C24.2, C25.2, C26.2, C27.2, C28.2, C29.2, C30.2, R6.1, R7.1, R8.1, R9.1, U2.16 (VDD33), U2.34 (VDD33), U2.52 (VDD33), U2.63 (VDD33); no longer J1.1
- net 5V: now also J5.18 (+5V), R1.1, C3.1, R2.1
- net CC1: now also R28.2
- net CC2: now also R29.2
- net HDMI_CLK_N: now also J5.12 (CK-)
- net HDMI_CLK_P: now also J5.10 (CK+)
- net HDMI_DATA0_N: now also J5.9 (D0-)
- net HDMI_DATA1_N: now also J5.6 (D1-)
- net HDMI_DATA1_P: now also J5.4 (D1+)
- net HDMI_DATA2_N: now also J5.3 (D2-)
- net HDMI_DATA2_P: now also J5.1 (D2+)
- net HDMI_HPD: now also J1.31, J5.19 (HPD), R1.2; no longer R1.1
- net HDMI_SCL: now also J5.15 (SCL)
- net HDMI_SDA: now also J5.16 (SDA)
- net LAN_BI_DC_N: now also J6.P8 (TD3-)
- net LAN_BI_DC_P: now also J6.P7 (TD3+)
- net LAN_BI_DD_N: now also J6.P10 (TD4-)
- net LAN_BI_DD_P: now also J6.P9 (TD4+)
- net LAN_LED: now also R20.2
- net LAN_RX_N: now also J6.P5 (TD2-)
- net LAN_RX_P: now also J6.P4 (TD2+)
- net LAN_TX_N: now also J6.P3 (TD1-)
- net LAN_TX_P: now also J6.P2 (TD1+)
- net USB0_3_RX_N: now also U2.7 (USB_SSRXM_DN1), USB1.5 (StdA_SSRX1-); no longer J1.54
- net USB0_3_RX_P: now also U2.6 (USB_SSRXP_DN1), USB1.6 (StdA_SSRX1+); no longer J1.55
- net USB0_3_TX_N: now also C4.2, U2.4 (USB_SSTXM_DN1); no longer J1.57
- net USB0_3_TX_P: now also C5.2, U2.3 (USB_SSTXP_DN1); no longer J1.58
- net USB0_N: now also U2.2 (USB_DM_DN1), USB1.2 (D1-); no longer J1.66
- net USB0_P: now also U2.1 (USB_DP_DN1), USB1.3 (D1+); no longer J1.67
- net USB1_N: now also U2.10 (USB_DM_DN2), USB1.11 (D2-)
- net USB1_P: now also U2.9 (USB_DP_DN2), USB1.12 (D2+)
- net USB2_N: now also U2.18 (USB_DM_DN3), USB2.2 (D1-)
- net USB2_P: now also U2.17 (USB_DP_DN3), USB2.3 (D1+)
- net GND: now reaches U1.2 (GND), U1.25 (GND)
- net GND: now also J1.47, J1.48, J1.53, J1.56, J1.59, J1.62, J1.65, J1.68, J1.75, J1.76, J1.77, J1.78, J1.79, J1.80, J2.A1 (GND), J2.A12 (GND), J2.B1 (GND), J2.B12 (GND), J2.S1 (SHIELD), J5.17 (GND), J5.SH, C10.2, C11.2, C12.1, C13.1, C14.1, C15.1, C20.1, C21.1, C22.1, C23.1, C24.1, C25.1, C26.1, C27.1, C28.1, C29.1, C3.2, C30.1, C31.1, C32.1, C33.1, C34.1, C35.1, C36.1, C37.1, C38.2, C39.2, C40.2, C41.2, C42.2, C43.2, C44.2, C45.2, C46.2, C47.2, C48.2, C49.1, C56.2, C57.2, C58.1, C8.1, C9.1, H1.1, H2.1, J6.P1 (GND), J6.S1 (SHIELD), J6.S2 (SHIELD__1), J8.1 (GND), R10.2, R11.2, R14.2, R15.2, R16.2, R18.1, R19.1, R26.2, R28.1, R29.1, R3.2, R32.2, R4.1, R5.1, U2.65 (VSS), U3.1 (GND), U3.11 (PAD), U4.1 (GND), U4.11 (PAD)
- net at U1.5 (VIO): now also C47.1, C48.1
- net at U1.6 (VDD): now also C46.1
- net USB_UART_5V: now reaches U1.7 (VREGIN)
- net HDMI_DATA0_P: now reaches J5.7 (D0+)
- net 12V renamed 12V_VOUT
- net 12V_VOUT: now also C51.1, C52.1, C53.1, C54.1, L1.2, R24.1
- new net: C60.2, R31.1
- new net: R31.2, U6.24 (PHASE)
- new net: C51.2, C52.2, C53.2, C54.2
- new net: C22.2, R17.1, Y1.2
- new net: C21.2, R17.2, Y1.1
- new net: L1.1, U5.5 (SW), U5.6 (SW), U5.7 (SW), U5.8 (SW), U5.9 (SW)
- new net: R18.2, U4.7 (ILM)
- new net: R23.1, U5.20 (MODE2)
- new net: C61.2, C62.2, C63.2, C64.2
- new net: C16.1, USB2.8 (StdA_SSTX1-)
- new net: R4.2, U2.40 (FULLPWRMGMTz/SMBA1/SS_UP)
- new net: R2.2, R3.1, U2.48 (USB_VBUS)
- new net: C55.1, U5.23 (BOOT)
- new net: C55.2, R27.1
- new net: R27.2, U5.24 (PHASE)
- new net: R30.1, U6.20 (MODE2)
- new net: R32.1, R33.2, U6.17 (FB)
- new net: R5.2, U2.42 (GANGED/SMBA2/HS_UP)
- new net: R16.1, U2.45 (AUTOENz/HS_SUSPEND)
- new net: R15.1, U2.49 (TEST)
- new net: C20.2, U2.50 (GRSTz)
- new net: C1.2, U2.55 (USB_SSTXP_UP)
- new net: C2.2, U2.56 (USB_SSTXM_UP)
- new net: R14.1, U2.64 (USB_R1)
- new net: R25.1, U5.14 (P_{GOOD})
- new net: R24.2, R26.1, U5.17 (FB)
- new net: J6.L3, R20.1
- new net: R19.2, U3.7 (ILM)
- new net: C59.1, U6.12 (V_{DRV})
- new net: C59.2, U6.13 (P_{GND}), U6.16 (A_{GND}), U6.25 (A_{GND}), U6.27 (P_{GND}), U6.3 (P_{GND}), U6.4 (P_{GND})
- new net: C4.1, USB1.8 (StdA_SSTX1-)
- new net: C18.1, USB2.17 (StdA_SSTX2-)
- new net: USB1.13 (GND2), USB1.16 (GND_DRAIN2), USB1.4 (GND1), USB1.7 (GND_DRAIN1)
- new net: C6.1, USB1.17 (StdA_SSTX2-)
- new net: C7.1, USB1.18 (StdA_SSTX2+)
- new net: C5.1, USB1.9 (StdA_SSTX1+)
- new net: C17.1, USB2.9 (StdA_SSTX1+)
- new net: C50.1, U5.12 (V_{DRV})
- new net: C50.2, U5.13 (P_{GND}), U5.16 (A_{GND}), U5.25 (A_{GND}), U5.27 (P_{GND}), U5.3 (P_{GND}), U5.4 (P_{GND})
- new net: J6.L1, R21.1
- new net: R22.1, U5.21 (MODE1)
- new net: U5.10 (GL), U5.11 (GL), U5.28 (GL)
- new net: L2.1, U6.5 (SW), U6.6 (SW), U6.7 (SW), U6.8 (SW), U6.9 (SW)
- new net: R13.1, U6.21 (MODE1)
- new net: R12.1, U6.14 (P_{GOOD})
- new net: C19.1, USB2.18 (StdA_SSTX2+)
- new net: U6.10 (GL), U6.11 (GL), U6.28 (GL)
- new net: C60.1, U6.23 (BOOT)
- new net: USB2.13 (GND2), USB2.16 (GND_DRAIN2), USB2.4 (GND1), USB2.7 (GND_DRAIN1)
- new net 1V1: C31.2, C32.2, C33.2, C34.2, C35.2, U2.13 (VDD), U2.21 (VDD), U2.28 (VDD), U2.31 (VDD), U2.5 (VDD), U2.51 (VDD), U2.57 (VDD), U2.8 (VDD)
- new net 20V: C10.1, C11.1, C56.1, C57.1, C58.2, C9.2, J8.2 (V+), U5.1 (V_{IN}), U5.2 (V_{IN}), U5.22 (V_{IN}), U5.26 (V_{IN}), U6.1 (V_{IN}), U6.2 (V_{IN}), U6.22 (V_{IN}), U6.26 (V_{IN})
- new net 5V_USB_0: C42.1, C43.1, U3.9 (OUT1), USB1.1 (VBUS1)
- new net 5V_USB_1: C44.1, C45.1, U3.8 (OUT2), USB1.10 (VBUS2)
- new net 5V_USB_2: C38.1, C39.1, U4.9 (OUT1), USB2.1 (VBUS1)
- new net 5V_USB_3: C40.1, C41.1, U4.8 (OUT2), USB2.10 (VBUS2)
- new net 5V_VOUT: C36.2, C37.2, C61.1, C62.1, C63.1, C64.1, L2.2, R33.1, U3.2 (IN), U3.3 (IN), U4.2 (IN), U4.3 (IN)
- new net BATEN0: R6.2, U2.36 (PWRCTL1/BATEN1), U3.4 (EN1)
- new net BATEN1: R7.2, U2.35 (PWRCTL2/BATEN2), U3.5 (EN2)
- new net BATEN2: R8.2, U2.33 (PWRCTL3/BATEN3), U4.4 (EN1)
- new net BATEN3: R9.2, U2.32 (PWRCTL4/BATEN4), U4.5 (EN2)
- new net EN: U5.19 (EN), U6.19 (EN)
- new net LAN_3V3: J1.1, J6.L2, J6.L4
- new net LED_1000: R21.2
- new net OVERCURRENT0: U2.46 (OVERCUR1z), U3.10 (~{FAULT1})
- new net OVERCURRENT1: U2.47 (OVERCUR2z), U3.6 (~{FAULT2})
- new net OVERCURRENT2: U2.44 (OVERCUR3z), U4.10 (~{FAULT1})
- new net OVERCURRENT3: U2.43 (OVERCUR4z), U4.6 (~{FAULT2})
- new net PGOOD: C49.2, C8.2, R12.2, R13.2, R22.2, R23.2, R25.2, R30.2, U5.15 (V_{DD}), U6.15 (V_{DD})
- new net PW_DC_SIGNAL: J8.4 (SIGNAL)
- new net SHIELD0: C12.2, C13.2, R10.1, USB1.19 (Shield), USB1.20 (Shield), USB1.21 (Shield), USB1.22 (Shield)
- new net SHIELD1: C14.2, C15.2, R11.1, USB2.19 (Shield), USB2.20 (Shield), USB2.21 (Shield), USB2.22 (Shield)
- new net USB1_3_RX_N: U2.15 (USB_SSRXM_DN2), USB1.14 (StdA_SSRX2-)
- new net USB1_3_RX_P: U2.14 (USB_SSRXP_DN2), USB1.15 (StdA_SSRX2+)
- new net USB1_3_TX_N: C6.2, U2.12 (USB_SSTXM_DN2)
- new net USB1_3_TX_P: C7.2, U2.11 (USB_SSTXP_DN2)
- new net USB2_3_RX_N: U2.23 (USB_SSRXM_DN3), USB2.5 (StdA_SSRX1-)
- new net USB2_3_RX_P: U2.22 (USB_SSRXP_DN3), USB2.6 (StdA_SSRX1+)
- new net USB2_3_TX_N: C16.2, U2.20 (USB_SSTXM_DN3)
- new net USB2_3_TX_P: C17.2, U2.19 (USB_SSTXP_DN3)
- new net USB3_3_RX_N: U2.30 (USB_SSRXM_DN4), USB2.14 (StdA_SSRX2-)
- new net USB3_3_RX_P: U2.29 (USB_SSRXP_DN4), USB2.15 (StdA_SSRX2+)
- new net USB3_3_TX_N: C18.2, U2.27 (USB_SSTXM_DN4)
- new net USB3_3_TX_P: C19.2, U2.26 (USB_SSTXP_DN4)
- new net USB3_N: U2.25 (USB_DM_DN4), USB2.11 (D2-)
- new net USB3_P: U2.24 (USB_DP_DN4), USB2.12 (D2+)
- new net USBUP_3_RX_N: J1.54, U2.59 (USB_SSRXM_UP)
- new net USBUP_3_RX_P: J1.55, U2.58 (USB_SSRXP_UP)
- new net USBUP_3_TX_N: C2.1, J1.57
- new net USBUP_3_TX_P: C1.1, J1.58
- new net USBUP_N: J1.66, U2.54 (USB_DM_UP)
- new net USBUP_P: J1.67, U2.53 (USB_DP_UP)
- new net XI_24: U2.61 (XO), U2.62 (XI)
- no-connect marks 3 -> 28
Other:
- note added: "0-20V @ 10A"
- note added: "CP2102 USB-UART"
- note added: "DC-Input"
- note added: "HDMI"
- note added: "Mounting holes"
- note added: "OPS connector"
- note added: "RJ45 GbE"
- note added: "TI USB8041 USB3.0 Hub"
- note added: "TPS2561 USB Power Switch (Port 0, 1)"
- note added: "TPS2561 USB Power Switch (Port 3, 4)"
- note added: "USB-C Debug"
- note added: "USB3.0 Port 0, 1"
- note added: "USB3.0 Port 2, 3"
- note added: "VIN 20V@5A"
- note added: "VOUT 12V@8A"
- note added: "VOUT 5V@8A"
- note added: "Vishay SiC438A (12V)"
- note added: "Vishay SiC438A (5V)"
- moved on the sheet: J1A, J1B, J2, J5, R1, U1
